File: futureKeyboardPCB/futureKeyboard/futureKeyboard.sch (KiCad schematic (older format))
At the start: 46 parts, among them P1 CONN_01X06, P3 CONN_01X02, Q1 2SC1815, Q2 2SC1815, SW1 SW_SPDT, SW2 SW_Push, SW3 SW_Push, SW4 SW_Push, SW5 SW_Push, U11 ESP32, U9 TA48033

Commit message: add right hand circuit on .sch file
Parts:
- removed C1, C2, C3, C5, C6: 0.1u, akizukit:SMD-2012, symbol Hyper_Board_Traser-rescue:C
- removed C4: 100u, Capacitor_THT:CP_Radial_D4.0mm_P2.00mm, symbol Hyper_Board_Traser-rescue:CP
- removed P1: CONN_01X06, Connector_PinHeader_2.54mm:PinHeader_1x06_P2.54mm_Vertical, symbol Hyper_Board_Traser-rescue:CONN_01X06
- removed P3: CONN_01X02, akizukit:Connector_EH_2pin, symbol Hyper_Board_Traser-rescue:CONN_01X02
- removed Q1, Q2: 2SC1815, Package_TO_SOT_THT:TO-92_Inline, symbol Transistor_BJT:2SC1815
- removed R17, R18, R19, R20, R21, R22, R26, R? (x5): 1k, akizukit:SMD-1608, symbol Hyper_Board_Traser-rescue:R
- removed R23, R?: 100, akizukit:SMD-1608, symbol Hyper_Board_Traser-rescue:R
- removed RV9, RV?: R_POT, akizukit:S_POT_SMD, symbol Device:R_POT
- removed SW1: SW_SPDT, Connector_PinHeader_2.54mm:PinHeader_1x03_P2.54mm_Vertical, symbol Switch:SW_SPDT
- removed SW2, SW3, SW4, SW5, SW? (x13): SW_Push, akizukit:SMD_SW, symbol Switch:SW_Push
- removed U11: ESP32, akizukit:ESP-WROOM-32, symbol akizukit:ESP32
- removed U9: TA48033, akizukit:AZ1086H, symbol Hyper_Board_Traser-rescue:TA48033
Connections:
- net labels removed: +3.3V, +3V3, +6V, DTR, EN, GND, IO0, RTS, RXD, TXD, back, c1, c2, c3, conv, enter, jx, jy, r1, r2, r3, r4
- wire segments 103 -> 0
- no-connect marks 22 -> 0
Other:
- note removed: "ROBOX_Writer"
- note removed: "joy stick"
- note removed: "left hand"
- note removed: "right hand"

Commit message: complete PCB
Parts:
- added J26, J27, J28, J29, J30, J31, J32, J33: Conn_01x01, akizukit:HOLE_3.2mm_nopad, symbol Connector_Generic:Conn_01x01
Connections:
- no-connect marks 0 -> 8
Changed lines of the file:
@@
 F1 "leftHand.sch" 50
 $EndSheet
+$Comp
+L Connector_Generic:Conn_01x01 J26
+U 1 1 5F5120C2
+P 2900 1150
+F 0 "J26" V 2772 1230 50  0000 L CNN
+F 1 "Conn_01x01" V 3000 950 50  0000 L CNN
+F 2 "akizukit:HOLE_3.2mm_nopad" H 2900 1150 50  0001 C CNN
+F 3 "~" H 2900 1150 50  0001 C CNN
+	1    2900 1150
+	0    1    1    0
+$EndComp
+$Comp
+L Connector_Generic:Conn_01x01 J27
+U 1 1 5F51214C
+P 2900 1550
+F 0 "J27" V 2772 1630 50  0000 L CNN
+F 1 "Conn_01x01" V 3000 1350 50  0000 L CNN
+F 2 "akizukit:HOLE_3.2mm_nopad" H 2900 1550 50  0001 C CNN
+F 3 "~" H 2900 1550 50  0001 C CNN
+	1    2900 1550
+	0    1    1    0
+$EndComp
+$Comp
+L Connector_Generic:Conn_01x01 J28
+U 1 1 5F512CC7
+P 3300 1150
+F 0 "J28" V 3172 1230 50  0000 L CNN
+F 1 "Conn_01x01" V 3400 950 50  0000 L CNN
+F 2 "akizukit:HOLE_3.2mm_nopad" H 3300 1150 50  0001 C CNN
+F 3 "~" H 3300 1150 50  0001 C CNN
+	1    3300 1150
+	0    1    1    0
+$EndComp
+$Comp
+L Connector_Generic:Conn_01x01 J29
+U 1 1 5F512CCD
+P 3300 1550
+F 0 "J29" V 3172 1630 50  0000 L CNN
+F 1 "Conn_01x01" V 3400 1350 50  0000 L CNN
+F 2 "akizukit:HOLE_3.2mm_nopad" H 3300 1550 50  0001 C CNN
+F 3 "~" H 3300 1550 50  0001 C CNN
+	1    3300 1550
+	0    1    1    0
+$EndComp
+$Comp
+L Connector_Generic:Conn_01x01 J30
+U 1 1 5F514CF5
+P 3700 1150
+F 0 "J30" V 3572 1230 50  0000 L CNN
+F 1 "Conn_01x01" V 3800 950 50  0000 L CNN
+F 2 "akizukit:HOLE_3.2mm_nopad" H 3700 1150 50  0001 C CNN
+F 3 "~" H 3700 1150 50  0001 C CNN
+	1    3700 1150
+	0    1    1    0
+$EndComp
+$Comp
+L Connector_Generic:Conn_01x01 J31
+U 1 1 5F514CFB
+P 3700 1550
+F 0 "J31" V 3572 1630 50  0000 L CNN
+F 1 "Conn_01x01" V 3800 1350 50  0000 L CNN
+F 2 "akizukit:HOLE_3.2mm_nopad" H 3700 1550 50  0001 C CNN
+F 3 "~" H 3700 1550 50  0001 C CNN
+	1    3700 1550
+	0    1    1    0
+$EndComp
+$Comp
+L Connector_Generic:Conn_01x01 J32
+U 1 1 5F514D01
+P 4100 1150
+F 0 "J32" V 3972 1230 50  0000 L CNN
+F 1 "Conn_01x01" V 4200 950 50  0000 L CNN
+F 2 "akizukit:HOLE_3.2mm_nopad" H 4100 1150 50  0001 C CNN
+F 3 "~" H 4100 1150 50  0001 C CNN
+	1    4100 1150
+	0    1    1    0
+$EndComp
+$Comp
+L Connector_Generic:Conn_01x01 J33
+U 1 1 5F514D07
+P 4100 1550
+F 0 "J33" V 3972 1630 50  0000 L CNN
+F 1 "Conn_01x01" V 4200 1350 50  0000 L CNN
+F 2 "akizukit:HOLE_3.2mm_nopad" H 4100 1550 50  0001 C CNN
+F 3 "~" H 4100 1550 50  0001 C CNN
+	1    4100 1550
+	0    1    1    0
+$EndComp
+NoConn ~ 2900 950
+NoConn ~ 2900 1350
+NoConn ~ 3300 1350
+NoConn ~ 3300 950
+NoConn ~ 3700 950
+NoConn ~ 4100 950
+NoConn ~ 4100 1350
+NoConn ~ 3700 1350
 $EndSCHEMATC
